File: PCB/Schematic/GPS/GPS_chip.sch (EAGLE design)
At the start: 7 parts, among them U1 VENUS638FLPX-L

Commit message: Updated GPS schematic
Replaced resistors, capacitors, and inductors with SMD packages.
Parts:
- C1, C2: device rcl:CPOL-USE1.8-4 -> rcl:C-USC0603
- L1: device rcl:L-US0204/5 -> rcl:L-USL4532P
- R1, R2: device rcl:R-EU_0204/5 -> rcl:R-US_R0603
Connections:
- net +3V3: now also C1.1; no longer C1.+
- net DGND: now also C1.2, C2.2; no longer C1.-, C2.-
- net N$2: now also C2.1; no longer C2.+
Changed lines of the file:
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@@
 <setting verticaltext="up"/>
 </settings>
-<grid distance="0.05" unitdist="inch" unit="inch" style="lines" multiple="1" display="no" altdistance="0.01" altunitdist="inch" altunit="inch"/>
+<grid distance="0.1" unitdist="inch" unit="inch" style="lines" multiple="1" display="no" altdistance="0.01" altunitdist="inch" altunit="inch"/>
 <layers>
 <layer number="1" name="Top" color="4" fill="1" visible="no" active="no"/>
@@
 <parts>
 <part name="U1" library="SparkFun-RF" deviceset="VENUS638FLPX-L" device=""/>
-<part name="C1" library="rcl" deviceset="CPOL-US" device="E1.8-4">
+<part name="C1" library="rcl" deviceset="C-US" device="C0603">
 <attribute name="CAP" value="0.1uF"/>
 </part>
 <part name="SUPPLY1" library="supply2" deviceset="DGND" device=""/>
 <part name="+3V1" library="supply1" deviceset="+3V3" device=""/>
-<part name="R1" library="rcl" deviceset="R-EU_" device="0204/5" value="4.7k"/>
+<part name="R1" library="rcl" deviceset="R-US_" device="R0603" value="4.7k"/>
 <part name="SUPPLY2" library="supply2" deviceset="AGND" device=""/>
 <part name="GND" library="supply2" deviceset="DGND" device=""/>
-<part name="L1" library="rcl" deviceset="L-US" device="0204/5" value="33nH"/>
+<part name="L1" library="rcl" deviceset="L-US" device="L4532P" value="33nH"/>
 <part name="ANT1" library="discrete" deviceset="ANTENNA" device=""/>
 <part name="+3V2" library="supply1" deviceset="+3V3" device=""/>
-<part name="R2" library="rcl" deviceset="R-EU_" device="0204/5" value="33k"/>
-<part name="C2" library="rcl" deviceset="CPOL-US" device="E1.8-4">
+<part name="R2" library="rcl" deviceset="R-US_" device="R0603" value="33k"/>
+<part name="C2" library="rcl" deviceset="C-US" device="C0603">
 <attribute name="CAP" value="0.1uF"/>
 </part>
@@
 </segment>
 <segment>
-<pinref part="C1" gate="G$1" pin="-"/>
+<pinref part="C1" gate="G$1" pin="2"/>
 <wire x1="-39.37" y1="58.42" x2="-39.37" y2="48.26" width="0.1524" layer="91"/>
 <pinref part="R1" gate="G$1" pin="1"/>
@@
 <wire x1="-54.61" y1="48.26" x2="-54.61" y2="46.99" width="0.1524" layer="91"/>
 <junction x="-39.37" y="48.26"/>
-<pinref part="C2" gate="G$1" pin="-"/>
+<pinref part="C2" gate="G$1" pin="2"/>
 <junction x="-29.21" y="48.26"/>
 </segment>
@@
 <wire x1="-29.21" y1="66.04" x2="-39.37" y2="66.04" width="0.1524" layer="91"/>
 <wire x1="-39.37" y1="66.04" x2="-39.37" y2="72.39" width="0.1524" layer="91"/>
-<pinref part="C1" gate="G$1" pin="+"/>
+<pinref part="C1" gate="G$1" pin="1"/>
 <junction x="-39.37" y="66.04"/>
 <pinref part="R2" gate="G$1" pin="2"/>
@@
 <pinref part="R2" gate="G$1" pin="1"/>
 <wire x1="-16.51" y1="55.88" x2="-29.21" y2="55.88" width="0.1524" layer="91"/>
-<pinref part="C2" gate="G$1" pin="+"/>
+<pinref part="C2" gate="G$1" pin="1"/>
 <junction x="-29.21" y="55.88"/>
 </segment>
